File: LoraHat.kicad_pcb (KiCad board)
At the start: 2 copper layers, 65.5 x 30.2 mm, 9 parts, among them J1-Raspberry1 Conn_02x20_Odd_Even

Commit message: V0.1
Parts:
- renumbered ESP32-WROOM-32D to MOD1, WIO-SX1262 to U2
Connections:
- J1-Raspberry1 pad 17: unconnected-(J1-Raspberry1-Pin_17-Pad17) -> +3.3V
- J1-Raspberry1 pad 2: +5V -> unconnected-(J1-Raspberry1-Pin_2-Pad2)
- J1-Raspberry1 pad 20: unconnected-(J1-Raspberry1-Pin_20-Pad20) -> GND
- J1-Raspberry1 pad 25: unconnected-(J1-Raspberry1-Pin_25-Pad25) -> GND
- J1-Raspberry1 pad 30: unconnected-(J1-Raspberry1-Pin_30-Pad30) -> GND
- J1-Raspberry1 pad 4: +5V -> unconnected-(J1-Raspberry1-Pin_4-Pad4)
- J1-Raspberry1 pad 9: unconnected-(J1-Raspberry1-Pin_9-Pad9) -> GND
Routing:
- net +3.3V: track 45.6 -> 32.2 mm, vias 2 -> 0
- net Net-(MOD1-IO16): track 27.3 -> 26.0 mm
- net Net-(MOD1-IO17): track 32.0 -> 31.2 mm
Other:
- board text added: "V0.1"
