File: LoraHat.kicad_sch (KiCad schematic)
At the start: 9 parts, among them J1-Raspberry1 Conn_02x20_Odd_Even, U2 Wio-SX1262

Commit message: V0.1
Connections:
- net +3.3V: now also J1-Raspberry1.17 (Pin_17)
- net GND: now also J1-Raspberry1.20 (Pin_20), J1-Raspberry1.25 (Pin_25), J1-Raspberry1.30 (Pin_30), J1-Raspberry1.9 (Pin_9)
- net +5V: no longer names the net of J1-Raspberry1.2 (Pin_2)
- net +5V: no longer J1-Raspberry1.4 (Pin_4)
Other:
- note added: "19/04/2026"
- note added: "João Uzêda"
- note added: "LoRa-Esp Raspberry Pi0 Hat"
